File: main-keyboard-pcb/main-keyboard-pcb.kicad_pcb (KiCad board)
At the start: 2 copper layers, 339.1 x 118.7 mm, 187 parts, among them J1 USB_B_Micro, J10 PF6, J11 PF7, J12 VCC, J13 D+, J14 D-, J15 GND, J2 MISO, J3 VCC, J4 SCK, J5 MOSI, J6 RES, J7 GND, J8 PF4, J9 PF5, Q1 NMOS, SW1 SW_Push, SW10 SW_Push, SW11 SW_Push, SW12 SW_Push, SW13 SW_Push, SW14 SW_Push, SW15 SW_Push, SW16 SW_Push, SW17 SW_Push, SW18 SW_Push, SW19 SW_Push, SW2 SW_Push, SW20 SW_Push, SW21 SW_Push, SW22 SW_Push, SW23 SW_Push, SW24 SW_Push, SW25 SW_Push, SW26 SW_Push, SW27 SW_Push, SW28 SW_Push, SW29 SW_Push, SW3 SW_Push, SW30 SW_Push, SW31 SW_Push, SW32 SW_Push, SW33 SW_Push, SW34 SW_Push, SW35 SW_Push, SW36 SW_Push, SW37 SW_Push, SW38 SW_Push, SW39 SW_Push, SW4 SW_Push, SW40 SW_Push, SW41 SW_Push, SW42 SW_Push, SW43 SW_Push, SW44 SW_Push, SW45 SW_Push, SW46 SW_Push, SW47 SW_Push, SW48 SW_Push, SW49 SW_Push, SW5 SW_Push, SW50 SW_Push, SW51 SW_Push, SW52 SW_Push, SW53 SW_Push, SW54 SW_Push, SW55 SW_Push, SW56 SW_Push, SW57 SW_Push, SW58 SW_Push, SW59 SW_Push, SW6 SW_Push, SW60 SW_Push, SW61 SW_Push, SW62 SW_Push, SW63 SW_Push, SW64 SW_Push, SW65 SW_Push, SW66 SW_Push, SW67 SW_Push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

Commit message: Removed old traces and routing
Parts:
- removed C1, C2: 22pF, Capacitors_SMD:C_0805_HandSoldering
- removed the C3 at (199.7, 87.1)
- removed C4: 1uF (±10%), Capacitors_SMD:C_0805_HandSoldering
- removed C5: 1uF, Capacitors_SMD:C_0805_HandSoldering
- removed C6, C7: 0.1uF, Capacitors_SMD:C_0805_HandSoldering
- removed the C8 at (183.9, 104.1)
- removed the C9 at (205.0, 92.9)
- removed G*** (x2): LOGO, arisu:arisu-logo
- removed J1: USB_B_Micro, Connectors_USB:USB_Micro-B_Molex-105017-0001
- removed J10: PF6, Pin_Headers:Pin_Header_Straight_1x01_Pitch2.54mm
- removed J11: PF7, Pin_Headers:Pin_Header_Straight_1x01_Pitch2.54mm
- removed J12, J3: VCC, Pin_Headers:Pin_Header_Straight_1x01_Pitch2.54mm
- removed J13: D+, Pin_Headers:Pin_Header_Straight_1x01_Pitch2.54mm
- removed J14: D-, Pin_Headers:Pin_Header_Straight_1x01_Pitch2.54mm
- removed J15, J7: GND, Pin_Headers:Pin_Header_Straight_1x01_Pitch2.54mm
- removed J2: MISO, Pin_Headers:Pin_Header_Straight_1x01_Pitch2.54mm
- removed J4: SCK, Pin_Headers:Pin_Header_Straight_1x01_Pitch2.54mm
- removed J5: MOSI, Pin_Headers:Pin_Header_Straight_1x01_Pitch2.54mm
- removed J6: RES, Pin_Headers:Pin_Header_Straight_1x01_Pitch2.54mm
- removed J8: PF4, Pin_Headers:Pin_Header_Straight_1x01_Pitch2.54mm
- removed J9: PF5, Pin_Headers:Pin_Header_Straight_1x01_Pitch2.54mm
- removed Q1: NMOS, buck-converter:BSS214NWH6327XTSA1
- removed the R1 at (177.3, 88.4)
- removed the R2 at (177.3, 86.3)
- removed R3, R4: 10K, Resistors_SMD:R_0805_HandSoldering
- removed SWR1: SW_Push, Buttons_Switches_SMD:SW_SPST_TL3342
- removed U1: SOIC127P600X175-8N, buck-converter:NE555D
- removed U1: USBLC6-2SC6, TO_SOT_Packages_SMD:SOT-23-6_Handsoldering
- removed the U2 at (192.1, 99.0)
- removed the Y1 at (209.8, 96.5)
- added IC1: LMR51420XDDCR, buck-converter:LMR51420XDDCR, F.Cu at (340.0, 50.1)
- C3: value 10nF -> 4.7uF
- C8: value 1.25uF -> C_Small
- C9: value 1nF -> 20uF
- D1: value 430mV -> D
- L1: value 22uH -> 25uH
- R1: value 1k -> 100k
- R2: value 1k -> 22.2k
- moved U2 176.1 mm to (190.5, 91.4)
Connections:
- net Net-(R1-Pad2) renamed BUCK_FB
- C3 pad 1: Net-(C3-Pad1) -> +5V
- C8 pad 1: +3.3V -> BUCK_CB
- C8 pad 2: GND -> BUCK_SW
- C9 pad 1: Net-(C9-Pad1) -> Net-(C16-Pad1)
- D1 pad 1: Net-(D1-Pad1) -> /row0
- D1 pad 2: GND -> Net-(D1-Pad2)
- D1 pad 1: (no net) -> /row0
- D1 pad 2: (no net) -> Net-(D1-Pad2)
- D10 pad 1: (no net) -> /row0
- D10 pad 2: (no net) -> Net-(D10-Pad2)
- D11 pad 1: (no net) -> /row1
- D11 pad 2: (no net) -> Net-(D11-Pad2)
- D12 pad 1: (no net) -> /row2
- D12 pad 2: (no net) -> Net-(D12-Pad2)
- D13 pad 1: (no net) -> /row3
- D13 pad 2: (no net) -> Net-(D13-Pad2)
- D14 pad 1: (no net) -> /row4
- D14 pad 2: (no net) -> Net-(D14-Pad2)
- D15 pad 1: (no net) -> /row0
- D15 pad 2: (no net) -> Net-(D15-Pad2)
- D16 pad 1: (no net) -> /row1
- D16 pad 2: (no net) -> Net-(D16-Pad2)
- D17 pad 1: (no net) -> /row2
- D17 pad 2: (no net) -> Net-(D17-Pad2)
- D18 pad 1: (no net) -> /row3
- D18 pad 2: (no net) -> Net-(D18-Pad2)
- D19 pad 1: (no net) -> /row0
- D19 pad 2: (no net) -> Net-(D19-Pad2)
- D2 pad 1: (no net) -> /row1
- D2 pad 2: (no net) -> Net-(D2-Pad2)
- D20 pad 1: (no net) -> /row1
- D20 pad 2: (no net) -> Net-(D20-Pad2)
- D21 pad 1: (no net) -> /row2
- D21 pad 2: (no net) -> Net-(D21-Pad2)
- D22 pad 1: (no net) -> /row3
- D22 pad 2: (no net) -> Net-(D22-Pad2)
- D23 pad 1: (no net) -> /row4
- D23 pad 2: (no net) -> Net-(D23-Pad2)
- D24 pad 1: (no net) -> /row0
- D24 pad 2: (no net) -> Net-(D24-Pad2)
- D25 pad 1: (no net) -> /row1
- D25 pad 2: (no net) -> Net-(D25-Pad2)
- D26 pad 1: (no net) -> /row2
- D26 pad 2: (no net) -> Net-(D26-Pad2)
- D27 pad 1: (no net) -> /row3
- D27 pad 2: (no net) -> Net-(D27-Pad2)
- D28 pad 1: (no net) -> /row4
- D28 pad 2: (no net) -> Net-(D28-Pad2)
- D29 pad 1: (no net) -> /row0
- D29 pad 2: (no net) -> Net-(D29-Pad2)
- D3 pad 1: (no net) -> /row2
- D3 pad 2: (no net) -> Net-(D3-Pad2)
- D30 pad 1: (no net) -> /row1
- D30 pad 2: (no net) -> Net-(D30-Pad2)
- D31 pad 1: (no net) -> /row2
- D31 pad 2: (no net) -> Net-(D31-Pad2)
- D32 pad 1: (no net) -> /row3
- D32 pad 2: (no net) -> Net-(D32-Pad2)
- D33 pad 1: (no net) -> /row0
- D33 pad 2: (no net) -> Net-(D33-Pad2)
- D34 pad 1: (no net) -> /row1
- D34 pad 2: (no net) -> Net-(D34-Pad2)
- D35 pad 1: (no net) -> /row2
- D35 pad 2: (no net) -> Net-(D35-Pad2)
- D36 pad 1: (no net) -> /row3
- D36 pad 2: (no net) -> Net-(D36-Pad2)
- D37 pad 1: (no net) -> /row4
- D37 pad 2: (no net) -> Net-(D37-Pad2)
- D38 pad 1: (no net) -> /row0
- D38 pad 2: (no net) -> Net-(D38-Pad2)
- D39 pad 1: (no net) -> /row1
- D39 pad 2: (no net) -> Net-(D39-Pad2)
- D4 pad 1: (no net) -> /row3
- D4 pad 2: (no net) -> Net-(D4-Pad2)
- D40 pad 1: (no net) -> /row2
- D40 pad 2: (no net) -> Net-(D40-Pad2)
- D41 pad 1: (no net) -> /row3
- D41 pad 2: (no net) -> Net-(D41-Pad2)
- D42 pad 1: (no net) -> /row0
- D42 pad 2: (no net) -> Net-(D42-Pad2)
- D43 pad 1: (no net) -> /row1
- D43 pad 2: (no net) -> Net-(D43-Pad2)
- D44 pad 1: (no net) -> /row2
- D44 pad 2: (no net) -> Net-(D44-Pad2)
- D45 pad 1: (no net) -> /row3
- D45 pad 2: (no net) -> Net-(D45-Pad2)
- D46 pad 1: (no net) -> /row4
- D46 pad 2: (no net) -> Net-(D46-Pad2)
- D47 pad 1: (no net) -> /row0
- D47 pad 2: (no net) -> Net-(D47-Pad2)
- D48 pad 1: (no net) -> /row1
- D48 pad 2: (no net) -> Net-(D48-Pad2)
- D49 pad 1: (no net) -> /row2
- D49 pad 2: (no net) -> Net-(D49-Pad2)
- D5 pad 1: (no net) -> /row4
- D5 pad 2: (no net) -> Net-(D5-Pad2)
- D50 pad 1: (no net) -> /row3
- D50 pad 2: (no net) -> Net-(D50-Pad2)
- D51 pad 1: (no net) -> /row0
- D51 pad 2: (no net) -> Net-(D51-Pad2)
- D52 pad 1: (no net) -> /row1
- D52 pad 2: (no net) -> Net-(D52-Pad2)
- D53 pad 1: (no net) -> /row2
- D53 pad 2: (no net) -> Net-(D53-Pad2)
- D54 pad 1: (no net) -> /row3
- D54 pad 2: (no net) -> Net-(D54-Pad2)
- D55 pad 1: (no net) -> /row0
- D55 pad 2: (no net) -> Net-(D55-Pad2)
- D56 pad 1: (no net) -> /row1
- D56 pad 2: (no net) -> Net-(D56-Pad2)
- D57 pad 1: (no net) -> /row2
- D57 pad 2: (no net) -> Net-(D57-Pad2)
- D58 pad 1: (no net) -> /row4
- D58 pad 2: (no net) -> Net-(D58-Pad2)
- D59 pad 1: (no net) -> /row0
- D59 pad 2: (no net) -> Net-(D59-Pad2)
- D6 pad 1: (no net) -> /row0
- D6 pad 2: (no net) -> Net-(D6-Pad2)
- D60 pad 1: (no net) -> /row1
- D60 pad 2: (no net) -> Net-(D60-Pad2)
- D61 pad 1: (no net) -> /row3
- D61 pad 2: (no net) -> Net-(D61-Pad2)
- D62 pad 1: (no net) -> /row4
- D62 pad 2: (no net) -> Net-(D62-Pad2)
- D63 pad 1: (no net) -> /row0
- D63 pad 2: (no net) -> Net-(D63-Pad2)
- D64 pad 1: (no net) -> /row1
- D64 pad 2: (no net) -> Net-(D64-Pad2)
- D65 pad 1: (no net) -> /row2
- D65 pad 2: (no net) -> Net-(D65-Pad2)
- D66 pad 1: (no net) -> /row3
- D66 pad 2: (no net) -> Net-(D66-Pad2)
- D67 pad 1: (no net) -> /row4
- D67 pad 2: (no net) -> Net-(D67-Pad2)
- D7 pad 1: (no net) -> /row1
- D7 pad 2: (no net) -> Net-(D7-Pad2)
- D8 pad 1: (no net) -> /row2
- D8 pad 2: (no net) -> Net-(D8-Pad2)
- D9 pad 1: (no net) -> /row3
- D9 pad 2: (no net) -> Net-(D9-Pad2)
- L1 pad 1: Net-(D1-Pad1) -> BUCK_SW
- L1 pad 2: +3.3V -> Net-(C16-Pad1)
- R1 pad 1: +5V -> Net-(C16-Pad1)
- R2 pad 2: Net-(C9-Pad1) -> GND
- SW1 pad 1: (no net) -> /col0
- SW1 pad 2: (no net) -> Net-(D1-Pad2)
- SW10 pad 1: (no net) -> /col2
- SW10 pad 2: (no net) -> Net-(D10-Pad2)
- SW11 pad 1: (no net) -> /col2
- SW11 pad 2: (no net) -> Net-(D11-Pad2)
- SW12 pad 1: (no net) -> /col2
- SW12 pad 2: (no net) -> Net-(D12-Pad2)
- SW13 pad 1: (no net) -> /col2
- SW13 pad 2: (no net) -> Net-(D13-Pad2)
- SW14 pad 1: (no net) -> /col2
- SW14 pad 2: (no net) -> Net-(D14-Pad2)
- SW15 pad 1: (no net) -> /col3
- SW15 pad 2: (no net) -> Net-(D15-Pad2)
- SW16 pad 1: (no net) -> /col3
- SW16 pad 2: (no net) -> Net-(D16-Pad2)
- SW17 pad 1: (no net) -> /col3
- SW17 pad 2: (no net) -> Net-(D17-Pad2)
- SW18 pad 1: (no net) -> /col3
- SW18 pad 2: (no net) -> Net-(D18-Pad2)
- SW19 pad 1: (no net) -> /col4
- SW19 pad 2: (no net) -> Net-(D19-Pad2)
- SW2 pad 1: (no net) -> /col0
- SW2 pad 2: (no net) -> Net-(D2-Pad2)
- SW20 pad 1: (no net) -> /col4
- SW20 pad 2: (no net) -> Net-(D20-Pad2)
- SW21 pad 1: (no net) -> /col4
- SW21 pad 2: (no net) -> Net-(D21-Pad2)
- SW22 pad 1: (no net) -> /col4
- SW22 pad 2: (no net) -> Net-(D22-Pad2)
- SW23 pad 1: (no net) -> /col4
- SW23 pad 2: (no net) -> Net-(D23-Pad2)
- SW24 pad 1: (no net) -> /col5
- SW24 pad 2: (no net) -> Net-(D24-Pad2)
- SW25 pad 1: (no net) -> /col5
- SW25 pad 2: (no net) -> Net-(D25-Pad2)
- SW26 pad 1: (no net) -> /col5
- SW26 pad 2: (no net) -> Net-(D26-Pad2)
- SW27 pad 1: (no net) -> /col5
- SW27 pad 2: (no net) -> Net-(D27-Pad2)
- SW28 pad 1: (no net) -> /col5
- SW28 pad 2: (no net) -> Net-(D28-Pad2)
- SW29 pad 1: (no net) -> /col6
- SW29 pad 2: (no net) -> Net-(D29-Pad2)
- SW3 pad 1: (no net) -> /col0
- SW3 pad 2: (no net) -> Net-(D3-Pad2)
- SW30 pad 1: (no net) -> /col6
- SW30 pad 2: (no net) -> Net-(D30-Pad2)
- SW31 pad 1: (no net) -> /col6
- SW31 pad 2: (no net) -> Net-(D31-Pad2)
- SW32 pad 1: (no net) -> /col6
- SW32 pad 2: (no net) -> Net-(D32-Pad2)
- SW33 pad 1: (no net) -> /col7
- SW33 pad 2: (no net) -> Net-(D33-Pad2)
- SW34 pad 1: (no net) -> /col7
- SW34 pad 2: (no net) -> Net-(D34-Pad2)
- SW35 pad 1: (no net) -> /col7
- SW35 pad 2: (no net) -> Net-(D35-Pad2)
- SW36 pad 1: (no net) -> /col7
- SW36 pad 2: (no net) -> Net-(D36-Pad2)
- SW37 pad 1: (no net) -> /col7
- SW37 pad 2: (no net) -> Net-(D37-Pad2)
- SW38 pad 1: (no net) -> /col8
- SW38 pad 2: (no net) -> Net-(D38-Pad2)
- SW39 pad 1: (no net) -> /col8
- SW39 pad 2: (no net) -> Net-(D39-Pad2)
- SW4 pad 1: (no net) -> /col0
- SW4 pad 2: (no net) -> Net-(D4-Pad2)
- SW40 pad 1: (no net) -> /col8
- SW40 pad 2: (no net) -> Net-(D40-Pad2)
- SW41 pad 1: (no net) -> /col8
- SW41 pad 2: (no net) -> Net-(D41-Pad2)
- SW42 pad 1: (no net) -> /col9
- SW42 pad 2: (no net) -> Net-(D42-Pad2)
- SW43 pad 1: (no net) -> /col9
- SW43 pad 2: (no net) -> Net-(D43-Pad2)
- SW44 pad 1: (no net) -> /col9
- SW44 pad 2: (no net) -> Net-(D44-Pad2)
- SW45 pad 1: (no net) -> /col9
- SW45 pad 2: (no net) -> Net-(D45-Pad2)
- SW46 pad 1: (no net) -> /col9
- SW46 pad 2: (no net) -> Net-(D46-Pad2)
- SW47 pad 1: (no net) -> /col10
- SW47 pad 2: (no net) -> Net-(D47-Pad2)
- SW48 pad 1: (no net) -> /col10
- SW48 pad 2: (no net) -> Net-(D48-Pad2)
- SW49 pad 1: (no net) -> /col10
- SW49 pad 2: (no net) -> Net-(D49-Pad2)
- SW5 pad 1: (no net) -> /col0
- SW5 pad 2: (no net) -> Net-(D5-Pad2)
- SW50 pad 1: (no net) -> /col10
- SW50 pad 2: (no net) -> Net-(D50-Pad2)
- SW51 pad 1: (no net) -> /col11
- SW51 pad 2: (no net) -> Net-(D51-Pad2)
- SW52 pad 1: (no net) -> /col11
- SW52 pad 2: (no net) -> Net-(D52-Pad2)
- SW53 pad 1: (no net) -> /col11
- SW53 pad 2: (no net) -> Net-(D53-Pad2)
- SW54 pad 1: (no net) -> /col11
- SW54 pad 2: (no net) -> Net-(D54-Pad2)
- SW55 pad 1: (no net) -> /col12
- SW55 pad 2: (no net) -> Net-(D55-Pad2)
- SW56 pad 1: (no net) -> /col12
- SW56 pad 2: (no net) -> Net-(D56-Pad2)
- SW57 pad 1: (no net) -> /col12
- SW57 pad 2: (no net) -> Net-(D57-Pad2)
- SW58 pad 1: (no net) -> /col12
- SW58 pad 2: (no net) -> Net-(D58-Pad2)
- SW59 pad 1: (no net) -> /col13
- SW59 pad 2: (no net) -> Net-(D59-Pad2)
- SW6 pad 1: (no net) -> /col1
- SW6 pad 2: (no net) -> Net-(D6-Pad2)
- SW60 pad 1: (no net) -> /col13
- SW60 pad 2: (no net) -> Net-(D60-Pad2)
- SW61 pad 1: (no net) -> /col13
- SW61 pad 2: (no net) -> Net-(D61-Pad2)
- SW62 pad 1: (no net) -> /col13
- SW62 pad 2: (no net) -> Net-(D62-Pad2)
- SW63 pad 1: (no net) -> /col14
- SW63 pad 2: (no net) -> Net-(D63-Pad2)
- SW64 pad 1: (no net) -> /col14
- SW64 pad 2: (no net) -> Net-(D64-Pad2)
- SW65 pad 1: (no net) -> /col14
- SW65 pad 2: (no net) -> Net-(D65-Pad2)
- SW66 pad 1: (no net) -> /col14
- SW66 pad 2: (no net) -> Net-(D66-Pad2)
- SW67 pad 1: (no net) -> /col14
- SW67 pad 2: (no net) -> Net-(D67-Pad2)
- SW7 pad 1: (no net) -> /col1
- SW7 pad 2: (no net) -> Net-(D7-Pad2)
- SW8 pad 1: (no net) -> /col1
- SW8 pad 2: (no net) -> Net-(D8-Pad2)
- SW9 pad 1: (no net) -> /col1
- SW9 pad 2: (no net) -> Net-(D9-Pad2)
Routing:
- net (no net): track 2728.1 -> 0.00 mm, vias 17 -> 0
- net +3.3V: track 811.9 -> 0.00 mm, vias 5 -> 0
- net GND: track 707.3 -> 0.00 mm, vias 17 -> 0
- net unconnected-(U2-Pad18): track 328.0 -> 0.00 mm, vias 4 -> 0
- net unconnected-(U2-Pad26): track 174.7 -> 0.00 mm
- net unconnected-(U2-Pad29): track 152.2 -> 0.00 mm
- net unconnected-(U2-Pad41): track 124.1 -> 0.00 mm
- net unconnected-(U2-Pad40): track 105.0 -> 0.00 mm
- net unconnected-(U2-Pad1): track 88.2 -> 0.00 mm, vias 2 -> 0
- net unconnected-(U2-Pad32): track 67.8 -> 0.00 mm
- net unconnected-(U2-Pad9): track 67.3 -> 0.00 mm, vias 2 -> 0
- net OSC_IN: track 53.0 -> 0.00 mm, vias 2 -> 0
- net unconnected-(U2-Pad31): track 49.4 -> 0.00 mm
- net unconnected-(U2-Pad38): track 40.2 -> 0.00 mm, vias 1 -> 0
- net unconnected-(U2-Pad8): track 39.8 -> 0.00 mm
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Other:
- board text removed: "Fate Design Rev 1.1"

Commit message: Updated diodes
Parts:
- D1: footprint buck-converter:RBE1KA20ATR -> DIODES_KEEB_2:1N4148W-13-F
- D1, D10, D11, D12, D13, D14, D15, D16, D17, D18, D19, D2, D20, D21, D22, D23, D24, D25, D26, D27, D28, D29, D3, D30, D31, D32, D33, D34, D35, D36, D37, D38, D39, D4, D40, D41, D42, D43, D44, D45, D46, D47, D48, D49, D5, D50, D51, D52, D53, D54, D55, D56, D57, D58, D59, D6, D60, D61, D62, D63, D64, D65, D66, D67, D7, D8, D9: footprint Diodes_SMD:D_SOD-123 -> DIODES_KEEB_2:1N4148W-13-F

Commit message: Completed footprint library for main-keyboard and rough part placement
Parts:
- removed the D1 at (25.8, 38.5)
- added C1: 2.2uF, stm32f4_2:GRM155R61E225KE11D, F.Cu at (195.8, 102.1)
- added C10: 0.1uF, stm32f4_2:GRM022R61A104ME01L, F.Cu at (186.4, 102.1)
- added C11: 0.1uF, stm32f4_2:GRM022R61A104ME01L, F.Cu at (197.6, 101.9)
- added C12: 0.1uF, stm32f4_2:GRM022R61A104ME01L, F.Cu at (201.2, 86.9)
- added C13: 10pF, stm32f4_2:GRM0225C1C100FA03L, F.Cu at (179.2, 93.2)
- added C14: 0.1uF, stm32f4_2:GRM022R61A104ME01L, F.Cu at (186.0, 83.3)
- added C15: 10pF, stm32f4_2:GRM0225C1C100FA03L, F.Cu at (179.2, 87.7)
- added C16: 20uF, buck-converter:GRMJN7R61C206ME05D, F.Cu at (214.4, 96.5)
- added C17: 0.1uF, stm32f4_2:GRM022R61A104ME01L, F.Cu at (182.4, 97.5)
- added C2: 4.7uF, stm32f4_2:GRM188R61C475KAAJD, F.Cu at (183.1, 85.1)
- added C4: 2.2uF, stm32f4_2:GRM155R61E225KE11D, F.Cu at (201.4, 88.4)
- added C5: 0.1uF, stm32f4_2:GRM022R61A104ME01L, F.Cu at (182.4, 88.9)
- added C6: 0.1uF, stm32f4_2:GRM022R61A104ME01L, F.Cu at (182.4, 91.4)
- added C7: 0.1uF, stm32f4_2:GRM022R61A104ME01L, F.Cu at (182.4, 96.0)
- added J1: Debug SWD Connector, Connector_PinHeader_1.27mm:PinHeader_2x05_P1.27mm_Vertical_SMD, F.Cu at (158.1, 85.7)
- added J2: Hotplug, Connector_PinHeader_2.54mm:PinHeader_1x04_P2.54mm_Vertical, F.Cu at (167.7, 83.2)
- added J3: USB_B_Micro, stm32f4_2:USB307530A, F.Cu at (207.6, 84.5)
- added R3: 10k, stm32f4_2:ERJ-UP3F1002V, F.Cu at (145.5, 87.1)
- added R4: 1k, stm32f4_2:ERJ-UP3D1001V, F.Cu at (175.3, 90.3)
- added R5: 2.2k, stm32f4_2:ERJ-UP3F2201V, F.Cu at (168.9, 86.4)
- added R6: 2.2k, stm32f4_2:ERJ-UP3F2201V, F.Cu at (172.5, 86.4)
- added SW99: SW_SPDT, Button_Switch_SMD:SW_SPDT_PCM12, F.Cu at (145.4, 83.2)
- added U1: USBLC6-4SC6, Package_TO_SOT_SMD:SOT-23-6, F.Cu at (207.4, 90.8)
- C3: footprint buck-converter:0402ZC103KAT2A -> stm32f4_2:GRM188R61C475KAAJD
- C8: value C_Small -> 0.1uF; footprint buck-converter:C2012X7R1H155K125AC -> stm32f4_2:GRM022R61A104ME01L
- C9: footprint buck-converter:EMK021BJ102MK-W -> buck-converter:GRMJN7R61C206ME05D
- L1: value 25uH -> 15uH; footprint buck-converter:SRP1038WA220M -> buck-converter:SRP1265WA150M
- R1: footprint buck-converter:ERJ-UP3D1001V -> buck-converter:CHV1206AJW-104ELF
- R2: footprint buck-converter:ERJ-UP3D1001V -> buck-converter:ERJP08F2212V
- U2: footprint stm32f4_2:QFP50P1600X1600X160-100N -> Package_QFP:LQFP-100_14x14mm_P0.5mm
- moved C9 203.8 mm to (214.4, 94.7)
- moved C8 200.5 mm to (215.9, 82.0), turned to 180 degrees
- moved L1 194.8 mm to (227.3, 88.9)
- moved R1 189.5 mm to (212.7, 91.4), turned to 90 degrees
- moved R2 178.7 mm to (215.9, 90.2), turned to -90 degrees
- moved C3 167.7 mm to (210.3, 90.2), turned to -90 degrees
- moved Y1 143.2 mm to (179.2, 90.3)
- moved IC1 128.8 mm to (215.9, 84.3)
- moved U2 1.80 mm to (191.8, 92.7)
Connections:
- C9 pad 1: Net-(C16-Pad1) -> +3V3
- D1 pad 1: /row0 -> row0
- D10 pad 1: /row0 -> row0
- D11 pad 1: /row1 -> row1
- D12 pad 1: /row2 -> row2
- D13 pad 1: /row3 -> row3
- D14 pad 1: /row4 -> row4
- D15 pad 1: /row0 -> row0
- D16 pad 1: /row1 -> row1
- D17 pad 1: /row2 -> row2
- D18 pad 1: /row3 -> row3
- D19 pad 1: /row0 -> row0
- D2 pad 1: /row1 -> row1
- D20 pad 1: /row1 -> row1
- D21 pad 1: /row2 -> row2
- D22 pad 1: /row3 -> row3
- D23 pad 1: /row4 -> row4
- D24 pad 1: /row0 -> row0
- D25 pad 1: /row1 -> row1
- D26 pad 1: /row2 -> row2
- D27 pad 1: /row3 -> row3
- D28 pad 1: /row4 -> row4
- D29 pad 1: /row0 -> row0
- D3 pad 1: /row2 -> row2
- D30 pad 1: /row1 -> row1
- D31 pad 1: /row2 -> row2
- D32 pad 1: /row3 -> row3
- D33 pad 1: /row0 -> row0
- D34 pad 1: /row1 -> row1
- D35 pad 1: /row2 -> row2
- D36 pad 1: /row3 -> row3
- D37 pad 1: /row4 -> row4
- D38 pad 1: /row0 -> row0
- D39 pad 1: /row1 -> row1
- D4 pad 1: /row3 -> row3
- D40 pad 1: /row2 -> row2
- D41 pad 1: /row3 -> row3
- D42 pad 1: /row0 -> row0
- D43 pad 1: /row1 -> row1
- D44 pad 1: /row2 -> row2
- D45 pad 1: /row3 -> row3
- D46 pad 1: /row4 -> row4
- D47 pad 1: /row0 -> row0
- D48 pad 1: /row1 -> row1
- D49 pad 1: /row2 -> row2
- D5 pad 1: /row4 -> row4
- D50 pad 1: /row3 -> row3
- D51 pad 1: /row0 -> row0
- D52 pad 1: /row1 -> row1
- D53 pad 1: /row2 -> row2
- D54 pad 1: /row3 -> row3
- D55 pad 1: /row0 -> row0
- D56 pad 1: /row1 -> row1
- D57 pad 1: /row2 -> row2
- D58 pad 1: /row4 -> row4
- D59 pad 1: /row0 -> row0
- D6 pad 1: /row0 -> row0
- D60 pad 1: /row1 -> row1
- D61 pad 1: /row3 -> row3
- D62 pad 1: /row4 -> row4
- D63 pad 1: /row0 -> row0
- D64 pad 1: /row1 -> row1
- D65 pad 1: /row2 -> row2
- D66 pad 1: /row3 -> row3
- D67 pad 1: /row4 -> row4
- D7 pad 1: /row1 -> row1
- D8 pad 1: /row2 -> row2
- D9 pad 1: /row3 -> row3
- L1 pad 2: Net-(C16-Pad1) -> +3V3
- R1 pad 1: Net-(C16-Pad1) -> +3V3
- SW1 pad 1: /col0 -> col0
- SW10 pad 1: /col2 -> col2
- SW11 pad 1: /col2 -> col2
- SW12 pad 1: /col2 -> col2
- SW13 pad 1: /col2 -> col2
- SW14 pad 1: /col2 -> col2
- SW15 pad 1: /col3 -> col3
- SW16 pad 1: /col3 -> col3
- SW17 pad 1: /col3 -> col3
- SW18 pad 1: /col3 -> col3
- SW19 pad 1: /col4 -> col4
- SW2 pad 1: /col0 -> col0
- SW20 pad 1: /col4 -> col4
- SW21 pad 1: /col4 -> col4
- SW22 pad 1: /col4 -> col4
- SW23 pad 1: /col4 -> col4
- SW24 pad 1: /col5 -> col5
- SW25 pad 1: /col5 -> col5
- SW26 pad 1: /col5 -> col5
- SW27 pad 1: /col5 -> col5
- SW28 pad 1: /col5 -> col5
- SW29 pad 1: /col6 -> col6
- SW3 pad 1: /col0 -> col0
- SW30 pad 1: /col6 -> col6
- SW31 pad 1: /col6 -> col6
- SW32 pad 1: /col6 -> col6
- SW33 pad 1: /col7 -> col7
- SW34 pad 1: /col7 -> col7
- SW35 pad 1: /col7 -> col7
- SW36 pad 1: /col7 -> col7
- SW37 pad 1: /col7 -> col7
- SW38 pad 1: /col8 -> col8
- SW39 pad 1: /col8 -> col8
- SW4 pad 1: /col0 -> col0
- SW40 pad 1: /col8 -> col8
- SW41 pad 1: /col8 -> col8
- SW42 pad 1: /col9 -> col9
- SW43 pad 1: /col9 -> col9
- SW44 pad 1: /col9 -> col9
- SW45 pad 1: /col9 -> col9
- SW46 pad 1: /col9 -> col9
- SW47 pad 1: /col10 -> col10
- SW48 pad 1: /col10 -> col10
- SW49 pad 1: /col10 -> col10
- SW5 pad 1: /col0 -> col0
- SW50 pad 1: /col10 -> col10
- SW51 pad 1: /col11 -> col11
- SW52 pad 1: /col11 -> col11
- SW53 pad 1: /col11 -> col11
- SW54 pad 1: /col11 -> col11
- SW55 pad 1: /col12 -> col12
- SW56 pad 1: /col12 -> col12
- SW57 pad 1: /col12 -> col12
- SW58 pad 1: /col12 -> col12
- SW59 pad 1: /col13 -> col13
- SW6 pad 1: /col1 -> col1
- SW60 pad 1: /col13 -> col13
- SW61 pad 1: /col13 -> col13
- SW62 pad 1: /col13 -> col13
- SW63 pad 1: /col14 -> col14
- SW64 pad 1: /col14 -> col14
- SW65 pad 1: /col14 -> col14
- SW66 pad 1: /col14 -> col14
- SW67 pad 1: /col14 -> col14
- SW7 pad 1: /col1 -> col1
- SW8 pad 1: /col1 -> col1
- SW9 pad 1: /col1 -> col1
- U2 pad 1: unconnected-(U2-Pad1) -> row0
- U2 pad 100: +3.3V -> +3V3
- U2 pad 11: +3.3V -> +3V3
- U2 pad 19: +3.3V -> +3V3
- U2 pad 2: unconnected-(U2-Pad2) -> row1
- U2 pad 22: +3.3V -> +3V3
- U2 pad 28: +3.3V -> +3V3
- U2 pad 29: unconnected-(U2-Pad29) -> col0
- U2 pad 3: unconnected-(U2-Pad3) -> row2
- U2 pad 30: unconnected-(U2-Pad30) -> col1
- U2 pad 31: unconnected-(U2-Pad31) -> col2
- U2 pad 32: unconnected-(U2-Pad32) -> col3
- U2 pad 33: unconnected-(U2-Pad33) -> col4
- U2 pad 34: unconnected-(U2-Pad34) -> col5
- U2 pad 35: unconnected-(U2-Pad35) -> col6
- U2 pad 4: unconnected-(U2-Pad4) -> row3
- U2 pad 5: unconnected-(U2-Pad5) -> row4
- U2 pad 50: +3.3V -> +3V3
- U2 pad 51: unconnected-(U2-Pad51) -> col14
- U2 pad 52: unconnected-(U2-Pad52) -> col13
- U2 pad 53: unconnected-(U2-Pad53) -> col12
- U2 pad 54: unconnected-(U2-Pad54) -> col11
- U2 pad 55: unconnected-(U2-Pad55) -> col10
- U2 pad 56: unconnected-(U2-Pad56) -> col9
- U2 pad 57: unconnected-(U2-Pad57) -> col8
- U2 pad 58: unconnected-(U2-Pad58) -> col7
- U2 pad 6: +3.3V -> +3V3
- U2 pad 70: USB_DM -> USB_CONN_DM
- U2 pad 71: USB_DP -> USB_CONN_DP
- U2 pad 75: +3.3V -> +3V3
Other:
- copper layers 2 -> 4

Commit message: Initial routing for stm32f4 and keyswitch matrix
Parts:
- moved C11 1.63 mm to (198.9, 100.8), turned to -90 degrees
- moved J3 0.90 mm to (207.8, 83.6)
- moved C1 0.25 mm to (196.1, 102.1)
Routing:
- net row3: track 0.00 -> 344.5 mm, vias 0 -> 16
- net row2: track 0.00 -> 332.0 mm, vias 0 -> 28
- net row4: track 0.00 -> 326.8 mm
- net row1: track 0.00 -> 326.8 mm, vias 0 -> 28
- net row0: track 0.00 -> 292.5 mm, vias 0 -> 26
- net col14: track 0.00 -> 115.8 mm
- net col12: track 0.00 -> 100.4 mm
- net col13: track 0.00 -> 96.3 mm
- net col7: track 0.00 -> 88.9 mm
- net col5: track 0.00 -> 88.4 mm
- net col9: track 0.00 -> 87.4 mm
- net col4: track 0.00 -> 85.9 mm
- net col2: track 0.00 -> 85.2 mm
- net col0: track 0.00 -> 80.3 mm
- net col6: track 0.00 -> 76.9 mm
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- added copper zone on In2.Cu, net +3V3
- added copper zone on In1.Cu, net GND

Commit message: Routed keyswitch matrix to microcontroller
Routing:
- net col0: track 80.3 -> 226.9 mm, vias 0 -> 1
- net col14: track 115.8 -> 261.4 mm, vias 0 -> 1
- net col1: track 61.9 -> 190.2 mm, vias 0 -> 1
- net col13: track 96.3 -> 222.1 mm, vias 0 -> 1
- net row4: track 326.8 -> 440.2 mm, vias 0 -> 11
- net col2: track 85.2 -> 194.2 mm, vias 0 -> 1
- net col12: track 100.4 -> 209.2 mm, vias 0 -> 1
- net col3: track 65.6 -> 155.7 mm, vias 0 -> 1
- net row3: track 344.5 -> 430.8 mm, vias 16 -> 27
- net col11: track 75.2 -> 157.8 mm, vias 0 -> 1
- net row2: track 332.0 -> 401.4 mm, vias 28 -> 37
- net col4: track 85.9 -> 154.9 mm, vias 0 -> 1
- net col10: track 66.8 -> 131.7 mm, vias 0 -> 1
- net col5: track 88.4 -> 146.0 mm, vias 0 -> 1
- net row1: track 326.8 -> 380.1 mm, vias 28 -> 35
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