File: LCDPCB/LCDPCB.kicad_sch (KiCad schematic)
At the start: 29 parts, among them J1 Sockets, J2 Hot Plug, J3 Programming Header, J4 Conn_01x08_Male, J5 Conn_01x08_Male, SW1 SW_Push, U1 STM32F091RCT6, U2 LD1117S12TR_SOT223

Commit message: v2 lcd pcb
Parts:
- added R5, R6: 10, lib_file:10R, symbol Device:R
- C1, C10, C3, C4, C6, C7, C8, C9: footprint lib_file:CAPC3225X88N -> lib_file:.1uF
- C5: footprint lib_file:22uFC -> lib_file:22uF
- J3: footprint lib_file:programming header -> Connector_PinSocket_2.54mm:PinSocket_2x05_P2.54mm_Vertical
- R1, R2: footprint lib_file:100KR -> lib_file:100k
- R3: footprint lib_file:ERJUP3 -> lib_file:1k
- R4: footprint lib_file:5.1kR -> lib_file:5.1k
Connections:
- net 3VA is gone; now on net +3.3V: U1.13 (VDDA)
- net +5V: now also C2.1, C3.1, U2.3 (VI)
- net PA6: now also R5.1; no longer J2.2 (Pin_2)
- net PA7: now also R6.1; no longer J2.3 (Pin_3)
- net V3.3_IN: no longer names the net of J3.7 (Pin_7)
- net V3.3_IN: no longer J3.8 (Pin_8)
- new net: J2.3 (Pin_3), R6.2
- new net: J2.2 (Pin_2), R5.2
- no-connect marks 47 -> 49
